Commit message: some edits in urdf and goal_pub script

File: src/irb_120_arm/urdf/irb_120_arm.urdf (robot description, URDF)
Before this commit: robot irb_120_arm, 8 links, 7 joints
Joints:
- joint joint_5: limit lower=-2.094 upper=2.094 effort=30 velocity=3 -> lower=-1.094 upper=3.094 effort=30 velocity=3

Commit message: moveit setup file is added

File: src/irb_120_arm/urdf/irb_120_arm.urdf (robot description, URDF)
Before this commit: robot irb_120_arm, 8 links, 7 joints
Joints:
- joint joint_5: limit lower=-1.094 upper=3.094 effort=30 velocity=3 -> lower=-2.094 upper=2.094 effort=30 velocity=3; origin xyz=-0.1789 0 0 rpy=0 0 1.5708 -> xyz=-0.1789 0 0 rpy=0 0 0
